File: paxbadge2022.kicad_pcb (KiCad board)
At the start: 2 copper layers, 102 x 81.5 mm, 188 parts, among them J1 Conn_01x02, J2 USB_B_Micro, J3 ICSP, J5 ILI9341, J6 Micro_SD_Card, Q1 BSS84, Q2 BSS84, SW1 0x0, SW10 1x1, SW11 2x1, SW12 3x1, SW13 4x1, SW14 5x1, SW15 6x1, SW16 7x1, SW17 0x2, SW18 1x2, SW19 2x2, SW2 1x0, SW20 3x2, SW21 4x2, SW22 5x2, SW23 6x2, SW24 7x2, SW25 0x3, SW26 1x3, SW27 2x3, SW28 3x3, SW29 4x3, SW3 2x0, SW30 5x3, SW31 6x3, SW32 7x3, SW33 0x4, SW34 1x4, SW35 2x4, SW36 3x4, SW37 4x4, SW38 5x4, SW39 6x4, SW4 3x0, SW40 7x4, SW41 0x5, SW42 1x5, SW43 2x5, SW44 3x5, SW45 4x5, SW46 5x5, SW47 6x5, SW48 7x5, SW49 0x6, SW5 4x0, SW50 1x6, SW51 2x6, SW52 3x6, SW53 4x6, SW54 5x6, SW55 6x6, SW56 7x6, SW57 0x7, SW58 1x7, SW59 2x7, SW6 5x0, SW60 3x7, SW61 4x7, SW62 5x7, SW63 6x7, SW64 7x7, SW65 RESTORE, SW66 UP, SW67 DOWN, SW68 LEFT, SW69 RIGHT, SW7 6x0, SW70 FIRE, SW72 PWR, SW8 7x0, SW9 0x1, U1 ATmega328PB-A, U2 MCP73831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

Commit message: nightly commit
Parts:
- D10, D11, D12, D13, D14, D15, D16, D17, D18, D19, D20, D21, D22, D23, D24, D25, D26, D27, D28, D29, D30, D31, D32, D33, D34, D35, D36, D37, D38, D39, D4, D40, D41, D42, D43, D44, D45, D46, D47, D48, D49, D5, D50, D51, D52, D53, D54, D55, D56, D57, D58, D59, D6, D60, D61, D62, D63, D64, D65, D66, D67, D7, D8, D9: footprint Diode_SMD:D_SOD-323 -> Diode_SMD:D_SOD-323F
- moved R8 89.7 mm to (40.7, 87.5), turned to 90 degrees
- moved R7 88.8 mm to (41.7, 87.5), turned to 90 degrees
- moved C13 3.13 mm to (37.7, 87.5), turned to 90 degrees
- moved C10 1.25 mm to (39.7, 87.5), turned to 90 degrees
- moved C9 1.12 mm to (41.9, 85.0)
- moved C12 1.10 mm to (41.9, 86.0)
- moved C11 0.72 mm to (38.7, 87.5), turned to 90 degrees
Routing:
- net /USB_D-: track 3.15 -> 119.1 mm, vias 1 -> 5
- net /USB_D+: track 3.15 -> 118.2 mm, vias 1 -> 5
- net /USB_DN: track 102.4 -> 1.56 mm, vias 2 -> 0
- net /USB_DP: track 101.2 -> 1.36 mm, vias 2 -> 0
- net +3V3: track 274.8 -> 266.7 mm
- net /KSCL: track 114.4 -> 107.8 mm
- net /KSDA: track 115.6 -> 109.0 mm
- net /RESET: track 145.9 -> 142.8 mm
- net GND: track 80.0 -> 79.4 mm, vias 41 -> 40
- net +1V1: track 13.7 -> 13.1 mm

Commit message: adding keyboard ino, syncing kicad after first prototype fixes
Parts:
- removed Q2: BSS84, Package_TO_SOT_SMD:SOT-23
- removed R9: 10k, Resistor_SMD:R_0402_1005Metric
- added C19: 100n, Capacitor_SMD:C_0402_1005Metric, B.Cu at (41.3, 84.9)
- moved R10 29.0 mm to (75.3, 88.9), turned to 90 degrees
- moved J3 5.66 mm to (114.5, 66.6), turned to 180 degrees
- moved C16 3.40 mm to (41.1, 99.0), turned to -90 degrees
- moved R7 2.78 mm to (40.0, 85.3)
- moved R8 2.78 mm to (39.0, 85.3)
- moved R11 2.08 mm to (40.0, 100.5), turned to 180 degrees
- moved C8 1.72 mm to (39.8, 99.0)
- moved C9 1.44 mm to (43.3, 85.3), turned to 90 degrees
- moved R6 1.30 mm to (42.2, 98.5), turned to 90 degrees
- moved C5 1.23 mm to (120.8, 93.3)
- moved U3 1.23 mm to (120.8, 96.2)
- moved C14 1.22 mm to (36.7, 94.3), turned to -90 degrees
- moved C10 0.90 mm to (40.6, 87.5)
- moved C11 0.90 mm to (39.6, 87.5)
- moved C13 0.90 mm to (38.6, 87.5)
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- renumbered C19 to C20
Connections:
- D10 pad 1: /KROW6 -> /KCOL6
- D11 pad 1: /KROW7 -> /KCOL7
- D12 pad 1: /KROW0 -> /KCOL0
- D13 pad 1: /KROW1 -> /KCOL1
- D14 pad 1: /KROW2 -> /KCOL2
- D15 pad 1: /KROW3 -> /KCOL3
- D16 pad 1: /KROW4 -> /KCOL4
- D17 pad 1: /KROW5 -> /KCOL5
- D18 pad 1: /KROW6 -> /KCOL6
- D19 pad 1: /KROW7 -> /KCOL7
- D20 pad 1: /KROW0 -> /KCOL0
- D21 pad 1: /KROW1 -> /KCOL1
- D22 pad 1: /KROW2 -> /KCOL2
- D23 pad 1: /KROW3 -> /KCOL3
- D24 pad 1: /KROW4 -> /KCOL4
- D25 pad 1: /KROW5 -> /KCOL5
- D26 pad 1: /KROW6 -> /KCOL6
- D27 pad 1: /KROW7 -> /KCOL7
- D28 pad 1: /KROW0 -> /KCOL0
- D29 pad 1: /KROW1 -> /KCOL1
- D30 pad 1: /KROW2 -> /KCOL2
- D31 pad 1: /KROW3 -> /KCOL3
- D32 pad 1: /KROW4 -> /KCOL4
- D33 pad 1: /KROW5 -> /KCOL5
- D34 pad 1: /KROW6 -> /KCOL6
- D35 pad 1: /KROW7 -> /KCOL7
- D36 pad 1: /KROW0 -> /KCOL0
- D37 pad 1: /KROW1 -> /KCOL1
- D38 pad 1: /KROW2 -> /KCOL2
- D39 pad 1: /KROW3 -> /KCOL3
- D4 pad 1: /KROW0 -> /KCOL0
- D40 pad 1: /KROW4 -> /KCOL4
- D41 pad 1: /KROW5 -> /KCOL5
- D42 pad 1: /KROW6 -> /KCOL6
- D43 pad 1: /KROW7 -> /KCOL7
- D44 pad 1: /KROW0 -> /KCOL0
- D45 pad 1: /KROW1 -> /KCOL1
- D46 pad 1: /KROW2 -> /KCOL2
- D47 pad 1: /KROW3 -> /KCOL3
- D48 pad 1: /KROW4 -> /KCOL4
- D49 pad 1: /KROW5 -> /KCOL5
- D5 pad 1: /KROW1 -> /KCOL1
- D50 pad 1: /KROW6 -> /KCOL6
- D51 pad 1: /KROW7 -> /KCOL7
- D52 pad 1: /KROW0 -> /KCOL0
- D53 pad 1: /KROW1 -> /KCOL1
- D54 pad 1: /KROW2 -> /KCOL2
- D55 pad 1: /KROW3 -> /KCOL3
- D56 pad 1: /KROW4 -> /KCOL4
- D57 pad 1: /KROW5 -> /KCOL5
- D58 pad 1: /KROW6 -> /KCOL6
- D59 pad 1: /KROW7 -> /KCOL7
- D6 pad 1: /KROW2 -> /KCOL2
- D60 pad 1: /KROW0 -> /KCOL0
- D61 pad 1: /KROW1 -> /KCOL1
- D62 pad 1: /KROW2 -> /KCOL2
- D63 pad 1: /KROW3 -> /KCOL3
- D64 pad 1: /KROW4 -> /KCOL4
- D65 pad 1: /KROW5 -> /KCOL5
- D66 pad 1: /KROW6 -> /KCOL6
- D67 pad 1: /KROW7 -> /KCOL7
- D7 pad 1: /KROW3 -> /KCOL3
- D8 pad 1: /KROW4 -> /KCOL4
- D9 pad 1: /KROW5 -> /KCOL5
- J3 pad 1: /KROW3 -> GND
- J3 pad 2: Net-(C3-Pad1) -> /RESET
- J3 pad 3: /KROW2 -> /KCOL4
- J3 pad 4: /KROW4 -> /KCOL2
- J3 pad 5: /RESET -> Net-(C3-Pad1)
- J3 pad 6: GND -> /KCOL3
- R10 pad 2: Net-(Q2-Pad2) -> GND
- SW1 pad 2: /KCOL0 -> /KROW0
- SW10 pad 2: /KCOL1 -> /KROW1
- SW11 pad 2: /KCOL1 -> /KROW1
- SW12 pad 2: /KCOL1 -> /KROW1
- SW13 pad 2: /KCOL1 -> /KROW1
- SW14 pad 2: /KCOL1 -> /KROW1
- SW15 pad 2: /KCOL1 -> /KROW1
- SW16 pad 2: /KCOL1 -> /KROW1
- SW17 pad 2: /KCOL2 -> /KROW2
- SW18 pad 2: /KCOL2 -> /KROW2
- SW19 pad 2: /KCOL2 -> /KROW2
- SW2 pad 2: /KCOL0 -> /KROW0
- SW20 pad 2: /KCOL2 -> /KROW2
- SW21 pad 2: /KCOL2 -> /KROW2
- SW22 pad 2: /KCOL2 -> /KROW2
- SW23 pad 2: /KCOL2 -> /KROW2
- SW24 pad 2: /KCOL2 -> /KROW2
- SW25 pad 2: /KCOL3 -> /KROW3
- SW26 pad 2: /KCOL3 -> /KROW3
- SW27 pad 2: /KCOL3 -> /KROW3
- SW28 pad 2: /KCOL3 -> /KROW3
- SW29 pad 2: /KCOL3 -> /KROW3
- SW3 pad 2: /KCOL0 -> /KROW0
- SW30 pad 2: /KCOL3 -> /KROW3
- SW31 pad 2: /KCOL3 -> /KROW3
- SW32 pad 2: /KCOL3 -> /KROW3
- SW33 pad 2: /KCOL4 -> /KROW4
- SW34 pad 2: /KCOL4 -> /KROW4
- SW35 pad 2: /KCOL4 -> /KROW4
- SW36 pad 2: /KCOL4 -> /KROW4
- SW37 pad 2: /KCOL4 -> /KROW4
- SW38 pad 2: /KCOL4 -> /KROW4
- SW39 pad 2: /KCOL4 -> /KROW4
- SW4 pad 2: /KCOL0 -> /KROW0
- SW40 pad 2: /KCOL4 -> /KROW4
- SW41 pad 2: /KCOL5 -> /KROW5
- SW42 pad 2: /KCOL5 -> /KROW5
- SW43 pad 2: /KCOL5 -> /KROW5
- SW44 pad 2: /KCOL5 -> /KROW5
- SW45 pad 2: /KCOL5 -> /KROW5
- SW46 pad 2: /KCOL5 -> /KROW5
- SW47 pad 2: /KCOL5 -> /KROW5
- SW48 pad 2: /KCOL5 -> /KROW5
- SW49 pad 2: /KCOL6 -> /KROW6
- SW5 pad 2: /KCOL0 -> /KROW0
- SW50 pad 2: /KCOL6 -> /KROW6
- SW51 pad 2: /KCOL6 -> /KROW6
- SW52 pad 2: /KCOL6 -> /KROW6
- SW53 pad 2: /KCOL6 -> /KROW6
- SW54 pad 2: /KCOL6 -> /KROW6
- SW55 pad 2: /KCOL6 -> /KROW6
- SW56 pad 2: /KCOL6 -> /KROW6
- SW57 pad 2: /KCOL7 -> /KROW7
- SW58 pad 2: /KCOL7 -> /KROW7
- SW59 pad 2: /KCOL7 -> /KROW7
- SW6 pad 2: /KCOL0 -> /KROW0
- SW60 pad 2: /KCOL7 -> /KROW7
- SW61 pad 2: /KCOL7 -> /KROW7
- SW62 pad 2: /KCOL7 -> /KROW7
- SW63 pad 2: /KCOL7 -> /KROW7
- SW64 pad 2: /KCOL7 -> /KROW7
- SW7 pad 2: /KCOL0 -> /KROW0
- SW8 pad 2: /KCOL0 -> /KROW0
- SW9 pad 2: /KCOL1 -> /KROW1
- U1 pad 1: /KCOL4 -> /KROW4
- U1 pad 10: /KCOL1 -> /KROW1
- U1 pad 11: /KCOL0 -> /KROW0
- U1 pad 12: /KROW7 -> /KCOL7
- U1 pad 13: /KROW6 -> /KCOL6
- U1 pad 14: /KROW5 -> /KCOL5
- U1 pad 15: /KROW4 -> /KCOL4
- U1 pad 16: /KROW3 -> /KCOL3
- U1 pad 17: /KROW2 -> /KCOL2
- U1 pad 2: /KCOL3 -> /KROW3
- U1 pad 30: /KCOL7 -> /KROW7
- U1 pad 31: /KCOL6 -> /KROW6
- U1 pad 32: /KCOL5 -> /KROW5
- U1 pad 7: /KROW1 -> /KCOL1
- U1 pad 8: /KROW0 -> /KCOL0
- U1 pad 9: /KCOL2 -> /KROW2
- U3 pad 2: unconnected-(U3-Pad2) -> GND
- U3 pad 4: GND -> unconnected-(U3-Pad4)
- U5 pad 26: /RESET -> unconnected-(U5-Pad26)
Routing:
- net /KROW5: track 91.2 -> 211.9 mm, vias 0 -> 2
- net /KCOL5: track 211.9 -> 91.2 mm, vias 2 -> 0
- net /KROW6: track 90.1 -> 197.2 mm, vias 0 -> 2
- net /KCOL6: track 197.2 -> 90.1 mm, vias 2 -> 0
- net /RESET: track 142.8 -> 40.1 mm, vias 2 -> 1
- net /KROW4: track 115.7 -> 205.6 mm, vias 1 -> 2
- net /KCOL4: track 205.6 -> 115.7 mm, vias 2 -> 1
- net /KROW3: track 126.5 -> 213.0 mm
- net /KCOL3: track 213.0 -> 126.5 mm
- net /KROW7: track 122.0 -> 202.1 mm, vias 0 -> 2
- net /KCOL7: track 202.1 -> 122.0 mm, vias 2 -> 0
- net /KROW1: track 132.6 -> 209.8 mm
- net /KCOL1: track 209.8 -> 132.6 mm
- net /KROW2: track 151.8 -> 207.4 mm, vias 1 -> 2
- net /KCOL2: track 207.4 -> 151.8 mm, vias 2 -> 1
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