File: paxbadge2022.kicad_sch (KiCad schematic)
At the start: 191 parts, among them J1 Conn_01x02, J2 USB_B_Micro, J3 ICSP, J4 JOYSTICK, J5 ILI9341, J6 Micro_SD_Card, J7 C64_KBD, Q1 BSS84, Q2 BSS84, SW1 0x0, SW10 1x1, SW11 2x1, SW12 3x1, SW13 4x1, SW14 5x1, SW15 6x1, SW16 7x1, SW17 0x2, SW18 1x2, SW19 2x2, SW2 1x0, SW20 3x2, SW21 4x2, SW22 5x2, SW23 6x2, SW24 7x2, SW25 0x3, SW26 1x3, SW27 2x3, SW28 3x3, SW29 4x3, SW3 2x0, SW30 5x3, SW31 6x3, SW32 7x3, SW33 0x4, SW34 1x4, SW35 2x4, SW36 3x4, SW37 4x4, SW38 5x4, SW39 6x4, SW4 3x0, SW40 7x4, SW41 0x5, SW42 1x5, SW43 2x5, SW44 3x5, SW45 4x5, SW46 5x5, SW47 6x5, SW48 7x5, SW49 0x6, SW5 4x0, SW50 1x6, SW51 2x6, SW52 3x6, SW53 4x6, SW54 5x6, SW55 6x6, SW56 7x6, SW57 0x7, SW58 1x7, SW59 2x7, SW6 5x0, SW60 3x7, SW61 4x7, SW62 5x7, SW63 6x7, SW64 7x7, SW65 RESTORE, SW66 UP, SW67 DOWN, SW68 LEFT, SW69 RIGHT, SW7 6x0, SW70 FIRE, SW71 RESET, SW72 PWR, SW8 7x0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

Commit message: nightly commit
Parts:
- D10, D11, D12, D13, D14, D15, D16, D17, D18, D19, D20, D21, D22, D23, D24, D25, D26, D27, D28, D29, D30, D31, D32, D33, D34, D35, D36, D37, D38, D39, D4, D40, D41, D42, D43, D44, D45, D46, D47, D48, D49, D5, D50, D51, D52, D53, D54, D55, D56, D57, D58, D59, D6, D60, D61, D62, D63, D64, D65, D66, D67, D7, D8, D9: footprint Diode_SMD:D_SOD-323 -> Diode_SMD:D_SOD-323F

Commit message: adding keyboard ino, syncing kicad after first prototype fixes
Parts:
- removed Q2: BSS84, Package_TO_SOT_SMD:SOT-23, symbol Transistor_FET:BSS84
- removed R9: 10k, Resistor_SMD:R_0402_1005Metric, symbol Device:R_Small
- removed SW71: RESET, Button_Switch_THT:SW_Tactile_SPST_Angled_PTS645Vx39-2LFS, symbol Switch:SW_Push
- added C19: 100n, Capacitor_SMD:C_0402_1005Metric, symbol Device:C_Small
- renumbered C19 to C20
Connections:
- net +3V3: now also C19.1
- net GND: now also J3.1 (Pin_1), R10.2, U3.2 (GND), C19.2; no longer J3.6 (Pin_6), U3.4 (GND)
- net KCOL0: now also D12.1 (K), D20.1 (K), D28.1 (K), D36.1 (K), D4.1 (K), D44.1 (K), D52.1 (K), D60.1 (K), J7.20 (Pin_20), U1.8 (XTAL2/PB7); no longer J7.12 (Pin_12), SW1.2, SW2.2, SW3.2, SW4.2, SW5.2, SW6.2, SW7.2, SW8.2, U1.11 (PD7)
- net KCOL1: now also D13.1 (K), D21.1 (K), D29.1 (K), D37.1 (K), D45.1 (K), D5.1 (K), D53.1 (K), D61.1 (K), J7.19 (Pin_19), U1.7 (XTAL1/PB6); no longer J7.11 (Pin_11), SW10.2, SW11.2, SW12.2, SW13.2, SW14.2, SW15.2, SW16.2, SW9.2, U1.10 (PD6)
- net KCOL2: now also D14.1 (K), D22.1 (K), D30.1 (K), D38.1 (K), D46.1 (K), D54.1 (K), D6.1 (K), D62.1 (K), J3.4 (Pin_4), J7.18 (Pin_18), U1.17 (PB5); no longer J7.10 (Pin_10), SW17.2, SW18.2, SW19.2, SW20.2, SW21.2, SW22.2, SW23.2, SW24.2, U1.9 (PD5)
- net KCOL3: now also D15.1 (K), D23.1 (K), D31.1 (K), D39.1 (K), D47.1 (K), D55.1 (K), D63.1 (K), D7.1 (K), J3.6 (Pin_6), J7.17 (Pin_17), U1.16 (PB4); no longer J7.9 (Pin_9), SW25.2, SW26.2, SW27.2, SW28.2, SW29.2, SW30.2, SW31.2, SW32.2, U1.2 (PD4)
- net KCOL4: now also D16.1 (K), D24.1 (K), D32.1 (K), D40.1 (K), D48.1 (K), D56.1 (K), D64.1 (K), D8.1 (K), J3.3 (Pin_3), J7.16 (Pin_16), U1.15 (PB3); no longer J7.8 (Pin_8), SW33.2, SW34.2, SW35.2, SW36.2, SW37.2, SW38.2, SW39.2, SW40.2, U1.1 (PD3)
- net KCOL5: now also D17.1 (K), D25.1 (K), D33.1 (K), D41.1 (K), D49.1 (K), D57.1 (K), D65.1 (K), D9.1 (K), J7.15 (Pin_15), U1.14 (PB2); no longer J7.7 (Pin_7), SW41.2, SW42.2, SW43.2, SW44.2, SW45.2, SW46.2, SW47.2, SW48.2, U1.32 (PD2)
- net KCOL6: now also D10.1 (K), D18.1 (K), D26.1 (K), D34.1 (K), D42.1 (K), D50.1 (K), D58.1 (K), D66.1 (K), J7.14 (Pin_14), U1.13 (PB1); no longer J7.6 (Pin_6), SW49.2, SW50.2, SW51.2, SW52.2, SW53.2, SW54.2, SW55.2, SW56.2, U1.31 (PD1)
- net KCOL7: now also D11.1 (K), D19.1 (K), D27.1 (K), D35.1 (K), D43.1 (K), D51.1 (K), D59.1 (K), D67.1 (K), J7.13 (Pin_13), U1.12 (PB0); no longer J7.5 (Pin_5), SW57.2, SW58.2, SW59.2, SW60.2, SW61.2, SW62.2, SW63.2, SW64.2, U1.30 (PD0)
- net KROW0: now also J7.12 (Pin_12), SW1.2, SW2.2, SW3.2, SW4.2, SW5.2, SW6.2, SW7.2, SW8.2, U1.11 (PD7); no longer D12.1 (K), D20.1 (K), D28.1 (K), D36.1 (K), D4.1 (K), D44.1 (K), D52.1 (K), D60.1 (K), J7.20 (Pin_20), U1.8 (XTAL2/PB7)
- net KROW1: now also J7.11 (Pin_11), SW10.2, SW11.2, SW12.2, SW13.2, SW14.2, SW15.2, SW16.2, SW9.2, U1.10 (PD6); no longer D13.1 (K), D21.1 (K), D29.1 (K), D37.1 (K), D45.1 (K), D5.1 (K), D53.1 (K), D61.1 (K), J7.19 (Pin_19), U1.7 (XTAL1/PB6)
- net KROW2: now also J7.10 (Pin_10), SW17.2, SW18.2, SW19.2, SW20.2, SW21.2, SW22.2, SW23.2, SW24.2, U1.9 (PD5); no longer D14.1 (K), D22.1 (K), D30.1 (K), D38.1 (K), D46.1 (K), D54.1 (K), D6.1 (K), D62.1 (K), J3.3 (Pin_3), J7.18 (Pin_18), U1.17 (PB5)
- net KROW3: now also J7.9 (Pin_9), SW25.2, SW26.2, SW27.2, SW28.2, SW29.2, SW30.2, SW31.2, SW32.2, U1.2 (PD4); no longer D15.1 (K), D23.1 (K), D31.1 (K), D39.1 (K), D47.1 (K), D55.1 (K), D63.1 (K), D7.1 (K), J3.1 (Pin_1), J7.17 (Pin_17), U1.16 (PB4)
- net KROW4: now also J7.8 (Pin_8), SW33.2, SW34.2, SW35.2, SW36.2, SW37.2, SW38.2, SW39.2, SW40.2, U1.1 (PD3); no longer D16.1 (K), D24.1 (K), D32.1 (K), D40.1 (K), D48.1 (K), D56.1 (K), D64.1 (K), D8.1 (K), J3.4 (Pin_4), J7.16 (Pin_16), U1.15 (PB3)
- net KROW5: now also J7.7 (Pin_7), SW41.2, SW42.2, SW43.2, SW44.2, SW45.2, SW46.2, SW47.2, SW48.2, U1.32 (PD2); no longer D17.1 (K), D25.1 (K), D33.1 (K), D41.1 (K), D49.1 (K), D57.1 (K), D65.1 (K), D9.1 (K), J7.15 (Pin_15), U1.14 (PB2)
- net KROW6: now also J7.6 (Pin_6), SW49.2, SW50.2, SW51.2, SW52.2, SW53.2, SW54.2, SW55.2, SW56.2, U1.31 (PD1); no longer D10.1 (K), D18.1 (K), D26.1 (K), D34.1 (K), D42.1 (K), D50.1 (K), D58.1 (K), D66.1 (K), J7.14 (Pin_14), U1.13 (PB1)
- net KROW7: now also J7.5 (Pin_5), SW57.2, SW58.2, SW59.2, SW60.2, SW61.2, SW62.2, SW63.2, SW64.2, U1.30 (PD0); no longer D11.1 (K), D19.1 (K), D27.1 (K), D35.1 (K), D43.1 (K), D51.1 (K), D59.1 (K), D67.1 (K), J7.13 (Pin_13), U1.12 (PB0)
- net RESET: now also J3.2 (Pin_2); no longer J3.5 (Pin_5), U5.26 (RUN)
- net at C3.1, D3.1 (K), U1.18 (AVCC)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: now also J3.5 (Pin_5); no longer J3.2 (Pin_2)
- no-connect marks 35 -> 37
Other:
- note added: "*"
- note added: "+"
- note added: ","
- note added: "-"
- note added: "."
- note added: "/"
- note added: "0"
- note added: "1"
- note added: "2"
- note added: "3"
- note added: "4"
- note added: "5"
- note added: "6"
- note added: "7"
- note added: "8"
- note added: "9"
- note added: ":"
- note added: ";"
- note added: "="
- note added: "@"
- note added: "A"
- note added: "B"
- note added: "C"
- note added: "C="
- note added: "CTRL"
- note added: "D"
- note added: "DEL"
- note added: "E"
- note added: "F"
- note added: "F1"
- note added: "F3"
- note added: "F5"
- note added: "F7"
- note added: "G"
- note added: "H"
- note added: "HOME"
- note added: "I"
- note added: "J"
- note added: "K"
- note added: "L"
- note added: "L-SHIFT"
- note added: "L/R"
- note added: "LEFT"
- note added: "M"
- note added: "N"
- note added: "O"
- note added: "P"
- note added: "Q"
- note added: "R"
- note added: "R-SHIFT"
- note added: "RETURN"
- note added: "RUN/STOP"
- note added: "S"
- note added: "SPACE"
- note added: "T"
- note added: "U"
- note added: "U/D"
- note added: "UP"
- note added: "V"
- note added: "W"
- note added: "X"
- note added: "Y"
- note added: "Z"
- note added: "£"
- moved on the sheet: J3, R10, R5
