File: c64pico.kicad_pcb (KiCad board)
At the start: 2 copper layers, 102 x 81.5 mm, 97 parts, among them J3 ICSP, J5 ILI9341, J6 Micro_SD_Card, SW1 0x0, SW10 1x1, SW11 2x1, SW12 3x1, SW13 4x1, SW14 5x1, SW15 6x1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

Commit message: add bom and update readme
Parts:
- J5: value ILI9341 -> CF4240FH0R0-05-NH
- LS1: value Speaker -> CPT-9019S-SMT
- SW71: value PWR -> JS102011SAQN
