File: c64pico.kicad_sch (KiCad schematic)
At the start: 99 parts, among them J3 ICSP, J4 JOYSTICK, J5 ILI9341, J6 Micro_SD_Card, J7 C64_KBD, SW1 0x0, SW10 1x1, SW11 2x1, SW12 3x1, SW13 4x1, SW14 5x1, SW15 6x1, SW16 7x1, SW17 0x2, SW18 1x2, SW19 2x2, SW2 1x0, SW20 3x2, SW21 4x2, SW22 5x2, SW23 6x2, SW24 7x2, SW25 0x3, SW26 1x3, SW27 2x3, SW28 3x3, SW29 4x3, SW3 2x0, SW30 5x3, SW31 6x3, SW32 7x3, SW33 0x4, SW34 1x4, SW35 2x4, SW36 3x4, SW37 4x4, SW38 5x4, SW39 6x4, SW4 3x0, SW40 7x4, SW41 0x5, SW42 1x5, SW43 2x5, SW44 3x5, SW45 4x5, SW46 5x5, SW47 6x5, SW48 7x5, SW49 0x6, SW5 4x0, SW50 1x6, SW51 2x6, SW52 3x6, SW53 4x6, SW54 5x6, SW55 6x6, SW56 7x6, SW57 0x7, SW58 1x7, SW59 2x7, SW6 5x0, SW60 3x7, SW61 4x7, SW62 5x7, SW63 6x7, SW64 7x7, SW65 RESTORE, SW66 UP, SW67 DOWN, SW68 LEFT, SW69 RIGHT, SW7 6x0, SW70 FIRE, SW71 PWR, SW8 7x0, SW9 0x1, U1 ATmega328PB-A, U2 BQ24230RGTT, U3 Pico

Commit message: add bom and update readme
Parts:
- J5: value ILI9341 -> CF4240FH0R0-05-NH; URL (none) -> https://www.aliexpress.com/item/32837085500.html
- J6: URL (none) -> https://www.aliexpress.com/item/32837085500.html
- LS1: value Speaker -> CPT-9019S-SMT
- SW71: value PWR -> JS102011SAQN
Other:
- note added: "(optional)"
- note added: "All tac switches are PTS 647 SN70 SMTR2 LFS"
- note added: "TFT must be ILI9341 2.4", 240x320px resolution 40-pin, 0.5mm pitch"
Changed lines of the file:
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@@
     (stroke (width 0) (type default) (color 0 0 0 0))
   )
-  (polyline (pts (xy 252.73 108.585) (xy 13.335 108.585))
+  (polyline (pts (xy 256.54 108.585) (xy 13.335 108.585))
     (stroke (width 0) (type default) (color 0 0 0 0))
   )
@@
     (stroke (width 0) (type default) (color 0 0 0 0))
   )
-  (polyline (pts (xy 252.73 216.535) (xy 252.73 108.585))
+  (polyline (pts (xy 256.54 216.535) (xy 256.54 108.585))
     (stroke (width 0) (type default) (color 0 0 0 0))
   )
@@
     (stroke (width 0) (type default) (color 0 0 0 0))
   )
-  (polyline (pts (xy 13.335 216.535) (xy 252.73 216.535))
+  (polyline (pts (xy 13.335 216.535) (xy 256.54 216.535))
     (stroke (width 0) (type default) (color 0 0 0 0))
   )
@@
     (effects (font (size 1.27 1.27)) (justify left bottom))
   )
+  (text "All tac switches are\nPTS 647 SN70 SMTR2 LFS" (at 229.87 115.57 0)
+    (effects (font (size 1.27 1.27)) (justify left bottom))
+  )
   (text "D20" (at 76.835 153.035 0)
     (effects (font (size 1.27 1.27)) (justify left bottom))
@@
     (effects (font (size 1.27 1.27)) (justify left bottom))
   )
+  (text "TFT must be ILI9341\n2.4\", 240x320px resolution\n40-pin, 0.5mm pitch"
+    (at 367.03 33.02 0)
+    (effects (font (size 1.27 1.27)) (justify left bottom))
+  )
   (text "To prevent ICSP pushing 5v to other circuitry!\nThis diode will drop VCC to about 2.7v,\nso run using internal 8MHz clock"
     (at 29.845 116.205 0)
@@
     (effects (font (size 1.27 1.27)) (justify left bottom))
   )
+  (text "(optional)" (at 243.205 158.115 0)
+    (effects (font (size 1.27 1.27)) (justify left bottom))
+  )
   (text "P" (at 132.08 179.705 0)
     (effects (font (size 1.27 1.27)) (justify left bottom))
@@
     (effects (font (size 1.27 1.27)) (justify left bottom))
   )
+  (text "(optional)" (at 240.03 31.75 0)
+    (effects (font (size 1.27 1.27)) (justify left bottom))
+  )
   (text "," (at 160.02 180.34 0)
     (effects (font (size 1.27 1.27)) (justify left bottom))
@@
       (effects (font (size 1.27 1.27)) hide)
     )
+    (property "URL" "https://www.aliexpress.com/item/32837085500.html" (id 4) (at 284.48 80.645 0)
+      (effects (font (size 1.27 1.27)) hide)
+    )
     (pin "1")
     (pin "2")
@@
       (effects (font (size 1.27 1.27)) (justify right))
     )
-    (property "Value" "PWR" (id 1) (at 80.518 38.6966 90)
+    (property "Value" "JS102011SAQN" (id 1) (at 80.518 38.6966 90)
       (effects (font (size 1.27 1.27)) (justify right))
     )
@@
       (effects (font (size 1.27 1.27)) (justify left))
     )
-    (property "Value" "Speaker" (id 1) (at 290.068 34.2516 0)
+    (property "Value" "CPT-9019S-SMT" (id 1) (at 290.068 34.2516 0)
       (effects (font (size 1.27 1.27)) (justify left))
     )
@@
       (effects (font (size 1.27 1.27)) (justify left))
     )
-    (property "Value" "ILI9341" (id 1) (at 355.727 72.3516 0)
+    (property "Value" "CF4240FH0R0-05-NH" (id 1) (at 355.727 72.3516 0)
       (effects (font (size 1.27 1.27)) (justify left))
     )
@@
       (effects (font (size 1.27 1.27)) hide)
     )
+    (property "URL" "https://www.aliexpress.com/item/32837085500.html" (id 4) (at 353.695 69.215 0)
+      (effects (font (size 1.27 1.27)) hide)
+    )
     (pin "1")
     (pin "10")
@@
     )
     (path "/e93c1126-a9f2-49f9-82f4-a3a6705a2449"
-      (reference "J5") (unit 1) (value "ILI9341") (footprint "Silvestron Components:ILI9341")
+      (reference "J5") (unit 1) (value "CF4240FH0R0-05-NH") (footprint "Silvestron Components:ILI9341")
     )
     (path "/88fb3154-d4cc-4239-872e-809899babc84"
@@
     )
     (path "/cbe80542-794c-47bf-a75c-dbd0a8dd3555"
-      (reference "LS1") (unit 1) (value "Speaker") (footprint "Buzzer_Beeper:Buzzer_CUI_CPT-9019S-SMT")
+      (reference "LS1") (unit 1) (value "CPT-9019S-SMT") (footprint "Buzzer_Beeper:Buzzer_CUI_CPT-9019S-SMT")
     )
     (path "/166558d0-12d0-47f5-a61a-e733d2ed8ada"
@@
     )
     (path "/a14a0292-2676-4936-b0ee-b4e10a9a8fff"
-      (reference "SW71") (unit 1) (value "PWR") (footprint "Button_Switch_SMD:SW_SPDT_CK-JS102011SAQN")
+      (reference "SW71") (unit 1) (value "JS102011SAQN") (footprint "Button_Switch_SMD:SW_SPDT_CK-JS102011SAQN")
     )
     (path "/ef777ebc-65a6-4f02-9962-13c95d7b5f1f"
